File: hardware/tempo-bt/tempo-bt.kicad_sch (KiCad schematic)
At the start: 69 parts, among them J1 JSTPH, J2 USB_C_Receptacle_USB2.0, J3 IO Interfaces, J4 QWIIC_CONNECTORJS-1MM, J5 2x5 PTH ARM CORTEX DEBUG, Q1 DMP3125L-7, SW1 JS102011SAQN, SW2 PTS850, SW3 PTS850, SW4 RESET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

Commit message: Update Keystone Battery holder
Parts:
- B1: value CR1220 -> 1056TR; NOTES BATT HOLDER -> CR1220 Battery + Holder
Changed lines of the file:
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@@
 			)
 		)
-		(property "Value" "CR1220"
+		(property "Value" "1056TR"
 			(at 102.87 36.83 0)
 			(effects
@@
 				)
 				(justify left bottom)
+				(hide yes)
 			)
 		)
@@
 			)
 		)
-		(property "NOTES" "BATT HOLDER"
-			(at 100.33 41.91 0)
+		(property "NOTES" "CR1220 Battery + Holder"
+			(at 105.918 41.656 0)
 			(effects
 				(font
 					(size 1.27 1.27)
 				)
-				(hide yes)
 			)
 		)
